Commit message: slam

File: src/mowen_gazebo/urdf/mowen.urdf (robot description, URDF)
Before this commit: robot mowen, 9 links, 8 joints
Joints:
- joint back_left_joint: origin xyz=-0.079748 0.1454 0.048587 rpy=1.5708 0 0 -> xyz=-0.079748 0.1454 0.048587 rpy=0 0 0
- joint back_right_joint: origin xyz=-0.079777 -0.1454 0.048399 rpy=-1.5708 0 3.1416 -> xyz=-0.079777 -0.1454 0.048399 rpy=0 0 0
- joint front_left_joint: origin xyz=0.12727 0.1454 0.048572 rpy=1.5708 0 0 -> xyz=0.12727 0.1454 0.048572 rpy=0 0 0
- joint front_right_joint: origin xyz=0.12721 -0.1454 0.048603 rpy=-1.5708 0 3.1416 -> xyz=0.12721 -0.1454 0.048603 rpy=0 0 0
